Commit message: some changes

File: sumo_ros_ws/src/sumo_description/urdf/base_components.xacro (robot description, xacro)
@@ -26,9 +26,4 @@
     </inertial>
   </link>
-  <joint name="frame_joint" type="fixed">
-    <parent link="base_link"/>
-    <child link="frame_link"/>
-    <origin xyz="0 0 0" rpy="0 0 0"/>
-  </joint>
   <!-- ========================================== -->
   <!-- LIDAR & SERVO                              -->
@@ -57,5 +52,5 @@
   </link>
   <joint name="lidar_joint" type="fixed">
-    <parent link="base_link"/>
+    <parent link="frame_link"/>
     <child link="lidar_link"/>
     <origin xyz="0 0.093257 0.10115" rpy="0 0 0"/>
@@ -73,5 +68,5 @@
   </link>
   <joint name="servo_joint" type="fixed">
-    <parent link="base_link"/>
+    <parent link="frame_link"/>
     <child link="servo_link"/>
     <origin xyz="0 0 0" rpy="0 0 0"/>
@@ -136,5 +131,5 @@
   </link>
   <joint name="camera_joint" type="fixed">
-    <parent link="base_link"/>
+    <parent link="frame_link"/>
     <child link="camera_link"/>
     <origin xyz="${c0_x} ${c0_y} ${c0_z}" rpy="0 0 0"/>
@@ -164,5 +159,5 @@
   </link>
   <joint name="camera1_joint" type="fixed">
-    <parent link="base_link"/>
+    <parent link="frame_link"/>
     <child link="camera1_link"/>
     <origin xyz="${c1_x} ${c1_y} ${c1_z}" rpy="0 0 0"/>
@@ -192,5 +187,5 @@
   </link>
   <joint name="camera2_joint" type="fixed">
-    <parent link="base_link"/>
+    <parent link="frame_link"/>
     <child link="camera2_link"/>
     <origin xyz="${c2_x} ${c2_y} ${c2_z}" rpy="0 0 0"/>
@@ -220,5 +215,5 @@
   </link>
   <joint name="camera3_joint" type="fixed">
-    <parent link="base_link"/>
+    <parent link="frame_link"/>
     <child link="camera3_link"/>
     <origin xyz="${c3_x} ${c3_y} ${c3_z}" rpy="0 0 0"/>

File: sumo_ros_ws/src/sumo_description/urdf/main.xacro (robot description, xacro)
@@ -35,5 +35,5 @@
   <xacro:property name="w3_m_x" value="-0.12352"/> <xacro:property name="w3_m_y" value="-0.10955"/> <xacro:property name="w3_m_z" value="0.095"/>
   <!-- ========================================== -->
-  <!-- Cameras Joints             -->
+  <!-- Cameras Joints                             -->
   <!-- ========================================== -->
   <xacro:property name="c0_x" value="0.10098"/> <xacro:property name="c0_y" value="-0.11001"/> <xacro:property name="c0_z" value="-0.005098"/>
@@ -49,7 +49,11 @@
   <material name="black"><color rgba="0.05 0.05 0.05 1.0"/></material>
   <material name="blue"><color rgba="0.1 0.1 0.8 1.0"/></material>
-  <!-- Base Link -->
-  <link name="base_link"></link>
+  <!-- Footprint Link -->
   <link name="base_footprint_link"/>
+  <joint name="base_footprint_joint" type="fixed">
+    <parent link="base_footprint_link"/>
+    <child link="frame_link"/>
+    <origin xyz="0 0 0.095" rpy="0 0 0"/>
+  </joint>
   <!-- ========================================== -->
   <!-- INCLUDES FOR OTHER XACRO FILES             -->
@@ -58,8 +62,3 @@
   <xacro:include filename="motors_couplers.xacro"/>
   <xacro:include filename="wheels.xacro"/>
-  <joint name="base_footprint_joint" type="fixed">
-    <parent link="base_footprint_link"/>
-    <child link="base_link"/>
-    <origin xyz="0 0 0.095" rpy="0 0 0"/>
-  </joint>
 </robot>

File: sumo_ros_ws/src/sumo_description/urdf/motors_couplers.xacro (robot description, xacro)
@@ -4,5 +4,5 @@
   <!-- MOTORS                                     -->
   <!-- ========================================== -->
-<xacro:macro name="motor_properties" params="mesh_file origin_xyz">
+  <xacro:macro name="motor_properties" params="mesh_file origin_xyz">
     <collision>
       <origin xyz="${origin_xyz}" rpy="0 0 0"/>
@@ -31,5 +31,5 @@
   </link>
   <joint name="motor_joint" type="fixed">
-    <parent link="base_link"/>
+    <parent link="frame_link"/>
     <child link="motor_link"/>
     <origin xyz="${m0_j_x} ${m0_j_y} ${m0_j_z}" rpy="0 0 0"/>
@@ -45,5 +45,5 @@
   </link>
   <joint name="motor1_joint" type="fixed">
-    <parent link="base_link"/>
+    <parent link="frame_link"/>
     <child link="motor1_link"/>
     <origin xyz="${m1_j_x} ${m1_j_y} ${m1_j_z}" rpy="0 0 0"/>
@@ -59,5 +59,5 @@
   </link>
   <joint name="motor2_joint" type="fixed">
-    <parent link="base_link"/>
+    <parent link="frame_link"/>
     <child link="motor2_link"/>
     <origin xyz="${m2_j_x} ${m2_j_y} ${m2_j_z}" rpy="0 0 0"/>
@@ -73,5 +73,5 @@
   </link>
   <joint name="motor3_joint" type="fixed">
-    <parent link="base_link"/>
+    <parent link="frame_link"/>
     <child link="motor3_link"/>
     <origin xyz="${m3_j_x} ${m3_j_y} ${m3_j_z}" rpy="0 0 0"/>

Commit message: Camera added

File: sumo_ros_ws/src/sumo_description/urdf/base_components.xacro (robot description, xacro)
@@ -219,3 +219,86 @@
     <origin xyz="${c3_x} ${c3_y} ${c3_z}" rpy="0 0 0"/>
   </joint>
+<!-- ========================================== -->
+  <!-- SENSOR & OPTICAL LINKS                     -->
+  <!-- ========================================== -->
+<link name="camera0_sensor_link">
+    <visual>
+      <origin xyz="0 0 0" rpy="0 0 0"/>
+      <geometry>
+        <box size="0.03 0.03 0.03"/>
+      </geometry>
+      <material name="red"/>
+    </visual>
+  </link>
+  <joint name="camera0_sensor_joint" type="fixed">
+      <parent link="frame_link"/>
+      <child link="camera0_sensor_link"/>
+      <origin xyz="${c0_x} ${c0_y} ${c0_z}" rpy="0 0 ${-pi/4}"/>
+  </joint>
+  <link name="camera_link_optical"/>
+  <joint name="camera_optical_joint" type="fixed">
+      <parent link="camera0_sensor_link"/>
+      <child link="camera_link_optical"/>
+      <origin xyz="0 0 0" rpy="0 0 0"/>
+  </joint>
+<link name="camera1_sensor_link">
+    <visual>
+      <origin xyz="0 0 0" rpy="0 0 0"/>
+      <geometry>
+        <box size="0.03 0.03 0.03"/>
+      </geometry>
+      <material name="red"/>
+    </visual>
+  </link>
+  <joint name="camera1_sensor_joint" type="fixed">
+      <parent link="frame_link"/>
+      <child link="camera1_sensor_link"/>
+      <origin xyz="${c1_x} ${c1_y} ${c1_z}" rpy="0 0 ${(-pi/4) + pi}"/>
+  </joint>
+  <link name="camera1_link_optical"/>
+  <joint name="camera1_optical_joint" type="fixed">
+      <parent link="camera1_sensor_link"/>
+      <child link="camera1_link_optical"/>
+      <origin xyz="0 0 0" rpy="0 0 0"/>
+  </joint>
+  <link name="camera2_sensor_link">
+    <visual>
+      <origin xyz="0 0 0" rpy="0 0 0"/>
+      <geometry>
+        <box size="0.03 0.03 0.03"/>
+      </geometry>
+      <material name="red"/>
+    </visual>
+  </link>
+  <joint name="camera2_sensor_joint" type="fixed">
+      <parent link="frame_link"/>
+      <child link="camera2_sensor_link"/>
+      <origin xyz="${c2_x} ${c2_y} ${c2_z}" rpy="0 0 ${5*pi/4}"/>
+  </joint>
+  <link name="camera2_link_optical"/>
+  <joint name="camera2_optical_joint" type="fixed">
+      <parent link="camera2_sensor_link"/>
+      <child link="camera2_link_optical"/>
+      <origin xyz="0 0 0" rpy="0 0 ${-pi/2}"/>
+  </joint>
+    <link name="camera3_sensor_link">
+    <visual>
+      <origin xyz="0 0 0" rpy="0 0 0"/>
+      <geometry>
+        <box size="0.03 0.03 0.03"/>
+      </geometry>
+      <material name="red"/>
+    </visual>
+  </link>
+  <joint name="camera3_sensor_joint" type="fixed">
+      <parent link="frame_link"/>
+      <child link="camera3_sensor_link"/>
+      <origin xyz="${c3_x} ${c3_y} ${c3_z}" rpy="0 0 ${9*pi/4}"/>
+  </joint>
+  <link name="camera3_link_optical"/>
+  <joint name="camera3_optical_joint" type="fixed">
+      <parent link="camera3_sensor_link"/>
+      <child link="camera3_link_optical"/>
+      <origin xyz="0 0 0" rpy="0 0 ${-pi/2}"/>
+  </joint>
 </robot>

File: sumo_ros_ws/src/sumo_description/urdf/gazebo_plugins.xacro (robot description, xacro)
@@ -1,24 +1,23 @@
 <?xml version="1.0"?>
 <robot xmlns:xacro="http://ros.org/wiki/xacro">
-  <!-- 1. Differential Drive Plugin -->
+    <!-- Control each wheel joint velocity independently -->
     <gazebo>
-        <plugin filename="gz-sim-diff-drive-system" name="gz::sim::systems::DiffDrive">
-            <!-- Left Wheels -->
-            <left_joint>wheel1_joint</left_joint>
-            <left_joint>wheel2_joint</left_joint>
-            <!-- Right Wheels -->
-            <right_joint>wheel_joint</right_joint>
-            <right_joint>wheel3_joint</right_joint>
-            <!-- Kinematics -->
-            <wheel_separation>0.242</wheel_separation>
-            <wheel_radius>0.032</wheel_radius>
-            <topic>/cmd_vel</topic>
-            <odom_topic>/odom</odom_topic>
-            <frame_id>odom</frame_id>
-            <child_frame_id>base_footprint_link</child_frame_id>
-            <odom_publish_frequency>50</odom_publish_frequency>
+        <plugin filename="gz-sim-joint-controller-system" name="gz::sim::systems::JointController">
+            <joint_name>wheel3_joint</joint_name>
+            <topic>/wheel_bl_cmd</topic>
+        </plugin>
+        <plugin filename="gz-sim-joint-controller-system" name="gz::sim::systems::JointController">
+            <joint_name>wheel1_joint</joint_name>
+            <topic>/wheel_fl_cmd</topic>
+        </plugin>
+        <plugin filename="gz-sim-joint-controller-system" name="gz::sim::systems::JointController">
+            <joint_name>wheel_joint</joint_name>
+            <topic>/wheel_br_cmd</topic>
+        </plugin>
+        <plugin filename="gz-sim-joint-controller-system" name="gz::sim::systems::JointController">
+            <joint_name>wheel2_joint</joint_name>
+            <topic>/wheel_fr_cmd</topic>
         </plugin>
     </gazebo>
-    <!-- 2. Joint State Publisher Plugin -->
     <gazebo>
         <plugin filename="gz-sim-joint-state-publisher-system" name="gz::sim::systems::JointStatePublisher">
@@ -31,3 +30,44 @@
         </plugin>
     </gazebo>
+    <gazebo>
+        <plugin filename="gz-sim-sensors-system" name="gz::sim::systems::Sensors">
+            <render_engine>ogre2</render_engine>
+        </plugin>
+    </gazebo>
+    <!-- ========================================== -->
+    <!-- CAMERA PLUGIN MACRO                        -->
+    <!-- ========================================== -->
+    <xacro:macro name="gazebo_camera_plugin" params="link_name topic_name optical_frame">
+        <gazebo reference="${link_name}">
+            <sensor name="${link_name}_sensor" type="camera">
+                <camera>
+                    <horizontal_fov>1.3962634</horizontal_fov>
+                    <image>
+                        <width>640</width>
+                        <height>480</height>
+                        <format>R8G8B8</format>
+                    </image>
+                    <clip>
+                        <near>0.1</near>
+                        <far>15</far>
+                    </clip>
+                    <noise>
+                        <type>gaussian</type>
+                        <mean>0.0</mean>
+                        <stddev>0.007</stddev>
+                    </noise>
+                    <optical_frame_id>${optical_frame}</optical_frame_id>
+                    <camera_info_topic>${topic_name}/camera_info</camera_info_topic>
+                </camera>
+                <always_on>1</always_on>
+                <update_rate>20</update_rate>
+                <visualize>true</visualize>
+                <topic>${topic_name}/image_raw</topic>
+            </sensor>
+        </gazebo>
+    </xacro:macro>
+    <xacro:gazebo_camera_plugin link_name="camera0_sensor_link" topic_name="camera0" optical_frame="camera_link_optical"/>
+    <xacro:gazebo_camera_plugin link_name="camera1_sensor_link" topic_name="camera1" optical_frame="camera1_link_optical"/>
+    <xacro:gazebo_camera_plugin link_name="camera2_sensor_link" topic_name="camera2" optical_frame="camera2_link_optical"/>
+    <xacro:gazebo_camera_plugin link_name="camera3_sensor_link" topic_name="camera3" optical_frame="camera3_link_optical"/>
 </robot>

File: sumo_ros_ws/src/sumo_description/urdf/main.xacro (robot description, xacro)
@@ -6,4 +6,10 @@
   <xacro:property name="rot_angle" value="0.785"/> <!-- 45 degrees in radians -->
   <xacro:property name="rot_45" value="0.707106"/> <!-- cos(45) and sin(45) -->
+  <!-- Camera Yaws (in radians) -->
+  <!-- Front: 0, Left: 1.5708, Back: 3.1416, Right: -1.5708 -->
+  <xacro:property name="c0_yaw" value="0"/>       <!-- أمامي -->
+  <xacro:property name="c1_yaw" value="1.5708"/>  <!-- يسار -->
+  <xacro:property name="c2_yaw" value="1.5708"/>  <!-- خلفي -->
+  <xacro:property name="c3_yaw" value="-1.5708"/> <!-- يمين -->
   <!-- ========================================== -->
   <!-- MOTORS ABSOLUTE POSITIONS (JOINT ORIGINS)  -->

File: sumo_ros_ws/src/sumo_description/urdf/sumo.xacro (robot description, xacro)
@@ -1,4 +1,7 @@
 <?xml version="1.0"?>
 <robot name="sumo_robot_visual_test">
+  <!-- ========================================== -->
+  <!-- Just a Unit Test for all links -->
+  <!-- ========================================== -->
   <material name="grey"><color rgba="0.5 0.5 0.5 1.0"/></material>
   <material name="dark_grey"><color rgba="0.2 0.2 0.2 1.0"/></material>

File: sumo_ros_ws/src/sumo_description/urdf/wheels.xacro (robot description, xacro)
@@ -4,8 +4,9 @@
   <!-- WHEELS MACRO                               -->
   <!-- ========================================== -->
-  <xacro:macro name="wheel_properties" params="mesh_file wx_m wy_m wz_m">
+  <xacro:macro name="wheel_properties" params="wx_m wy_m wz_m rot">
     <collision>
-      <origin xyz="${(wx_m + wy_m) * rot_45} ${(-wx_m + wy_m) * rot_45} ${wz_m}" rpy="0 0 -${rot_angle}"/>
-      <geometry><mesh filename="package://sumo_description/meshes_fixed/${mesh_file}"/></geometry>
+      <origin xyz="${(wx_m + wy_m) * rot_45} ${(-wx_m + wy_m) * rot_45} ${wz_m}" rpy="0 1.5708 0"/>
+      <geometry><cylinder radius="0.038" length="0.03"/></geometry>
+      <!-- <geometry><mesh filename="package://sumo_description/meshes_fixed/Wheel.stl"/></geometry> -->
     </collision>
     <inertial>
@@ -21,42 +22,43 @@
     </inertial>
   </xacro:macro>
-  <!-- Wheel 0 -->
   <link name="wheel_link">
     <visual>
-      <origin xyz="${(w0_m_x + w0_m_y) * rot_45} ${(-w0_m_x + w0_m_y) * rot_45} ${w0_m_z}" rpy="0 0 -${rot_angle}"/>
+      <origin xyz="0 0 0" rpy="0 0 -${rot_angle + 1.5708}"/>
       <geometry><mesh filename="package://sumo_description/meshes_fixed/Wheel.stl"/></geometry>
       <material name="black"/>
     </visual>
-    <xacro:wheel_properties mesh_file="Wheel.stl" wx_m="${w0_m_x}" wy_m="${w0_m_y}" wz_m="${w0_m_z}"/>
+    <xacro:wheel_properties wx_m="0" wy_m="0" wz_m="0" rot="${2*rot_angle + 1.5708}"/>
   </link>
   <joint name="wheel_joint" type="continuous">
     <parent link="coupler_link"/>
     <child link="wheel_link"/>
-    <origin xyz="${c0_m_x - w0_m_x} ${c0_m_y - w0_m_y} ${c0_m_z - w0_m_z}" rpy="0 0 ${rot_angle}"/>
-    <axis xyz="0 1 0"/>
+    <origin xyz="${c0_m_x - w0_m_x} ${c0_m_y - w0_m_y} ${c0_m_z - w0_m_z}" rpy="0 0 ${rot_angle + 1.5708 + 3.14159}"/>
+    <axis xyz="1 0 0"/>
+    <dynamics damping="0.01" friction="0.01"/>
   </joint>
   <!-- Wheel 1 -->
   <link name="wheel1_link">
     <visual>
-      <origin xyz="${(w1_m_x + w1_m_y) * rot_45} ${(-w1_m_x + w1_m_y) * rot_45} ${w1_m_z}" rpy="0 0 -${rot_angle}"/>
+      <origin xyz="0 0 0" rpy="0 0 -${rot_angle+1.5708}"/>
       <geometry><mesh filename="package://sumo_description/meshes_fixed/Wheel1.stl"/></geometry>
       <material name="black"/>
     </visual>
-    <xacro:wheel_properties mesh_file="Wheel1.stl" wx_m="${w1_m_x}" wy_m="${w1_m_y}" wz_m="${w1_m_z}"/>
+    <xacro:wheel_properties wx_m="0" wy_m="0" wz_m="0" rot="${2*rot_angle+1.5708}"/>
   </link>
   <joint name="wheel1_joint" type="continuous">
     <parent link="coupler1_link"/>
     <child link="wheel1_link"/>
-    <origin xyz="${c1_m_x - w1_m_x} ${c1_m_y - w1_m_y} ${c1_m_z - w1_m_z}" rpy="0 0 ${rot_angle}"/>
-    <axis xyz="0 1 0"/>
+    <origin xyz="${c1_m_x - w1_m_x} ${c1_m_y - w1_m_y} ${c1_m_z - w1_m_z}" rpy="0 0 ${rot_angle+1.5708 + 3.14159}"/>
+    <axis xyz="1 0 0"/>
+    <dynamics damping="0.01" friction="0.01"/>
   </joint>
-  <!-- Wheel 2 -->
+  <!-- Wheel 2 (Original Working Axis X) -->
   <link name="wheel2_link">
     <visual>
-      <origin xyz="${(w2_m_x + w2_m_y) * rot_45} ${(-w2_m_x + w2_m_y) * rot_45} ${w2_m_z}" rpy="0 0 -${rot_angle}"/>
+      <origin xyz="0 0 0" rpy="0 0 -${rot_angle}"/>
       <geometry><mesh filename="package://sumo_description/meshes_fixed/Wheel2.stl"/></geometry>
       <material name="black"/>
     </visual>
-    <xacro:wheel_properties mesh_file="Wheel2.stl" wx_m="${w2_m_x}" wy_m="${w2_m_y}" wz_m="${w2_m_z}"/>
+    <xacro:wheel_properties wx_m="0" wy_m="0" wz_m="0" rot="${2*rot_angle+1.5708}"/>
   </link>
   <joint name="wheel2_joint" type="continuous">
@@ -65,13 +67,14 @@
     <origin xyz="${c2_m_x - w2_m_x} ${c2_m_y - w2_m_y} ${c2_m_z - w2_m_z}" rpy="0 0 ${rot_angle}"/>
     <axis xyz="1 0 0"/>
+    <dynamics damping="0.01" friction="0.01"/>
   </joint>
-  <!-- Wheel 3 -->
+  <!-- Wheel 3 (Original Working Axis X) -->
   <link name="wheel3_link">
     <visual>
-      <origin xyz="${(w3_m_x + w3_m_y) * rot_45} ${(-w3_m_x + w3_m_y) * rot_45} ${w3_m_z}" rpy="0 0 -${rot_angle}"/>
+      <origin xyz="0 0 0" rpy="0 0 -${rot_angle}"/>
       <geometry><mesh filename="package://sumo_description/meshes_fixed/Wheel3.stl"/></geometry>
       <material name="black"/>
     </visual>
-    <xacro:wheel_properties mesh_file="Wheel3.stl" wx_m="${w3_m_x}" wy_m="${w3_m_y}" wz_m="${w3_m_z}"/>
+    <xacro:wheel_properties wx_m="0" wy_m="0" wz_m="0" rot="${2*rot_angle+1.5708}"/>
   </link>
   <joint name="wheel3_joint" type="continuous">
@@ -80,4 +83,41 @@
     <origin xyz="${c3_m_x - w3_m_x} ${c3_m_y - w3_m_y} ${c3_m_z - w3_m_z}" rpy="0 0 ${rot_angle}"/>
     <axis xyz="1 0 0"/>
+    <dynamics damping="0.01" friction="0.01"/>
   </joint>
+  <gazebo reference="wheel_link">
+    <mu1>1.0</mu1>
+    <mu2>0.01</mu2>
+    <fdir1>0 1 0</fdir1>
+    <kp>1000000.0</kp>
+    <kd>100.0</kd>
+    <minDepth>0.001</minDepth>
+    <maxVel>0.1</maxVel>
+  </gazebo>
+  <gazebo reference="wheel1_link">
+    <mu1>1.0</mu1>
+    <mu2>0.01</mu2>
+    <fdir1>0 1 0</fdir1>
+    <kp>1000000.0</kp>
+    <kd>100.0</kd>
+    <minDepth>0.001</minDepth>
+    <maxVel>0.1</maxVel>
+  </gazebo>
+  <gazebo reference="wheel2_link">
+    <mu1>1.0</mu1>
+    <mu2>0.01</mu2>
+    <fdir1>0 1 0</fdir1>
+    <kp>1000000.0</kp>
+    <kd>100.0</kd>
+    <minDepth>0.001</minDepth>
+    <maxVel>0.1</maxVel>
+  </gazebo>
+  <gazebo reference="wheel3_link">
+    <mu1>1.0</mu1>
+    <mu2>0.01</mu2>
+    <fdir1>0 1 0</fdir1>
+    <kp>1000000.0</kp>
+    <kd>100.0</kd>
+    <minDepth>0.001</minDepth>
+    <maxVel>0.1</maxVel>
+  </gazebo>
 </robot>
